File: PCB/5V2_Supplies.sch (KiCad schematic (older format))
At the start: 52 parts, among them Q1 DMN6068LK3-13, Q2 DMN6068LK3-13, U15 RT7258GSP, U16 RT7258GSP, U4 TS462CDT

Commit message: Added ELOAD to sch and imported to layout
Parts:
- added J16, J17: Conn_01x03, Pin_Headers:Pin_Header_Straight_1x03_Pitch2.54mm_SMD_Pin1Right, symbol Conn_01x03
Connections:
- net 5V2_A: now also J17.1 (Pin_1), J17.2 (Pin_2)
- net 5V2_B: now also J16.1 (Pin_1), J16.2 (Pin_2)
- net GND: now also J16.3 (Pin_3), J17.3 (Pin_3)
