File: PCB/USB.sch (KiCad schematic (older format))
At the start: 23 parts, among them Q14 DMG1026UV-7, U8 CY7C65634-48AXCT, Y1 12MHz

Commit message: Added ELOAD to sch and imported to layout
Parts:
- removed Q14: DMG1026UV-7, digikey-footprints:SOT-563, symbol DMG1026UV-7
- added Q4: 2N7002, TO_SOT_Packages_SMD:SOT-23, symbol 2N7002
Connections:
- net GND: now also Q4.2 (S)
- net USB_RST: now also Q4.1 (G)
- net USB_VBUS_DET: now also Q4.3 (D)
Other:
- note removed: "Unused gate"
- moved on the sheet: R128
Changed lines of the file:
@@
 $Descr A 11000 8500
 encoding utf-8
-Sheet 7 11
+Sheet 7 12
 Title "USB"
 Date "2018-06-13"
-Rev "01"
+Rev "02"
 Comp ""
 Comment1 ""
@@
 $EndComp
 $Comp
-L GND #PWR0117
+L GND #PWR0120
 U 1 1 5B225E9F
 P 6850 1900
-F 0 "#PWR0117" H 6850 1650 50  0001 C CNN
+F 0 "#PWR0120" H 6850 1650 50  0001 C CNN
 F 1 "GND" H 6850 1750 50  0000 C CNN
 F 2 "" H 6850 1900 50  0001 C CNN
@@
 $EndComp
 $Comp
-L +3V3 #PWR0118
+L +3V3 #PWR0121
 U 1 1 5B226286
 P 6850 1050
-F 0 "#PWR0118" H 6850 900 50  0001 C CNN
+F 0 "#PWR0121" H 6850 900 50  0001 C CNN
 F 1 "+3V3" H 6850 1190 50  0000 C CNN
 F 2 "" H 6850 1050 50  0001 C CNN
@@
 $EndComp
 $Comp
-L GND #PWR0119
+L GND #PWR0122
 U 1 1 5B22826A
 P 1100 3950
-F 0 "#PWR0119" H 1100 3700 50  0001 C CNN
+F 0 "#PWR0122" H 1100 3700 50  0001 C CNN
 F 1 "GND" H 1100 3800 50  0000 C CNN
 F 2 "" H 1100 3950 50  0001 C CNN
@@
 $EndComp
 $Comp
-L GND #PWR0120
+L GND #PWR0123
 U 1 1 5B2282C0
 P 1850 3950
-F 0 "#PWR0120" H 1850 3700 50  0001 C CNN
+F 0 "#PWR0123" H 1850 3700 50  0001 C CNN
 F 1 "GND" H 1850 3800 50  0000 C CNN
 F 2 "" H 1850 3950 50  0001 C CNN
@@
 $EndComp
 $Comp
-L GND #PWR0121
+L GND #PWR0124
 U 1 1 5B227D9A
 P 8100 4200
-F 0 "#PWR0121" H 8100 3950 50  0001 C CNN
+F 0 "#PWR0124" H 8100 3950 50  0001 C CNN
 F 1 "GND" H 8100 4050 50  0000 C CNN
 F 2 "" H 8100 4200 50  0001 C CNN
@@
 $EndComp
 $Comp
-L GND #PWR0122
+L GND #PWR0125
 U 1 1 5B227E05
 P 8600 4200
-F 0 "#PWR0122" H 8600 3950 50  0001 C CNN
+F 0 "#PWR0125" H 8600 3950 50  0001 C CNN
 F 1 "GND" H 8600 4050 50  0000 C CNN
 F 2 "" H 8600 4200 50  0001 C CNN
@@
 $EndComp
 $Comp
-L +3V3 #PWR0123
+L +3V3 #PWR0126
 U 1 1 5B227F97
 P 8100 2700
-F 0 "#PWR0123" H 8100 2550 50  0001 C CNN
+F 0 "#PWR0126" H 8100 2550 50  0001 C CNN
 F 1 "+3V3" H 8100 2840 50  0000 C CNN
 F 2 "" H 8100 2700 50  0001 C CNN
@@
 $EndComp
 $Comp
-L +3V3 #PWR0124
+L +3V3 #PWR0127
 U 1 1 5B228002
 P 8600 2700
-F 0 "#PWR0124" H 8600 2550 50  0001 C CNN
+F 0 "#PWR0127" H 8600 2550 50  0001 C CNN
 F 1 "+3V3" H 8600 2840 50  0000 C CNN
 F 2 "" H 8600 2700 50  0001 C CNN
@@
 Text Notes 9050 3350 0    60   ~ 0
 Optional pullup / pulldowns \nfor unused port
-$Comp
-L DMG1026UV-7 Q14
-U 1 1 5B228C75
-P 2750 6250
-F 0 "Q14" H 2950 6325 50  0000 L CNN
-F 1 "DMG1026UV-7" H 2950 6250 50  0000 L CNN
-F 2 "digikey-footprints:SOT-563" H 2950 6175 50  0001 L CIN
-F 3 "" H 2750 6250 50  0001 L CNN
-	1    2750 6250
-	1    0    0    -1
-$EndComp
-Text GLabel 2200 6300 0    60   Input ~ 0
+Text GLabel 2200 6250 0    60   Input ~ 0
 USB_RST
 $Comp
-L GND #PWR0125
+L GND #PWR0128
 U 1 1 5B228DF5
 P 2850 6600
-F 0 "#PWR0125" H 2850 6350 50  0001 C CNN
+F 0 "#PWR0128" H 2850 6350 50  0001 C CNN
 F 1 "GND" H 2850 6450 50  0000 C CNN
 F 2 "" H 2850 6600 50  0001 C CNN
@@
 L R_Small R128
 U 1 1 5B2E84CE
-P 2350 6550
-F 0 "R128" H 2400 6600 50  0000 L CNN
-F 1 "10k" H 2400 6500 50  0000 L CNN
-F 2 "Resistors_SMD:R_0603" H 2350 6550 50  0001 C CNN
-F 3 "" H 2350 6550 50  0001 C CNN
-F 4 "0603" H 2500 6400 60  0000 C CNN "Package"
-	1    2350 6550
-	1    0    0    -1
-$EndComp
-$Comp
-L GND #PWR0126
+P 2350 6500
+F 0 "R128" H 2400 6550 50  0000 L CNN
+F 1 "10k" H 2400 6450 50  0000 L CNN
+F 2 "Resistors_SMD:R_0603" H 2350 6500 50  0001 C CNN
+F 3 "" H 2350 6500 50  0001 C CNN
+F 4 "0603" H 2500 6350 60  0000 C CNN "Package"
+	1    2350 6500
+	1    0    0    -1
+$EndComp
+$Comp
+L GND #PWR0129
 U 1 1 5B2E8600
-P 2350 6750
-F 0 "#PWR0126" H 2350 6500 50  0001 C CNN
-F 1 "GND" H 2350 6600 50  0000 C CNN
-F 2 "" H 2350 6750 50  0001 C CNN
-F 3 "" H 2350 6750 50  0001 C CNN
-	1    2350 6750
-	1    0    0    -1
-$EndComp
-$Comp
-L GND #PWR0127
+P 2350 6700
+F 0 "#PWR0129" H 2350 6450 50  0001 C CNN
+F 1 "GND" H 2350 6550 50  0000 C CNN
+F 2 "" H 2350 6700 50  0001 C CNN
+F 3 "" H 2350 6700 50  0001 C CNN
+	1    2350 6700
+	1    0    0    -1
+$EndComp
+$Comp
+L GND #PWR0130
 U 1 1 5B347A31
 P 5500 5650
-F 0 "#PWR0127" H 5500 5400 50  0001 C CNN
+F 0 "#PWR0130" H 5500 5400 50  0001 C CNN
 F 1 "GND" H 5500 5500 50  0000 C CNN
 F 2 "" H 5500 5650 50  0001 C CNN
@@
 $EndComp
 $Comp
-L +3V3 #PWR0128
+L +3V3 #PWR0131
 U 1 1 5B349BFC
 P 5600 1950
-F 0 "#PWR0128" H 5600 1800 50  0001 C CNN
+F 0 "#PWR0131" H 5600 1800 50  0001 C CNN
 F 1 "+3V3" H 5600 2090 50  0000 C CNN
 F 2 "" H 5600 1950 50  0001 C CNN
@@
 	1600 3400 1850 3400
 Wire Wire Line
-	2350 6750 2350 6650
-Wire Wire Line
-	2200 6300 2550 6300
-Wire Wire Line
-	2350 6450 2350 6300
-Connection ~ 2350 6300
+	2350 6700 2350 6600
+Wire Wire Line
+	2200 6250 2550 6250
+Wire Wire Line
+	2350 6400 2350 6250
+Connection ~ 2350 6250
 Wire Wire Line
 	5350 5300 5350 5450
@@
 $EndComp
 $Comp
-L +3V3 #PWR0129
+L +3V3 #PWR0132
 U 1 1 5B34D2A4
 P 2250 2400
-F 0 "#PWR0129" H 2250 2250 50  0001 C CNN
+F 0 "#PWR0132" H 2250 2250 50  0001 C CNN
 F 1 "+3V3" H 2250 2540 50  0000 C CNN
 F 2 "" H 2250 2400 50  0001 C CNN
@@
 $EndComp
 $Comp
-L +3V3 #PWR0130
+L +3V3 #PWR0133
 U 1 1 5B34D31F
 P 2650 2400
-F 0 "#PWR0130" H 2650 2250 50  0001 C CNN
+F 0 "#PWR0133" H 2650 2250 50  0001 C CNN
 F 1 "+3V3" H 2650 2540 50  0000 C CNN
 F 2 "" H 2650 2400 50  0001 C CNN
@@
 $EndComp
 $Comp
-L +3V3 #PWR0131
+L +3V3 #PWR0134
 U 1 1 5B34D37E
 P 3050 2400
-F 0 "#PWR0131" H 3050 2250 50  0001 C CNN
+F 0 "#PWR0134" H 3050 2250 50  0001 C CNN
 F 1 "+3V3" H 3050 2540 50  0000 C CNN
 F 2 "" H 3050 2400 50  0001 C CNN
@@
 	3050 3400 4400 3400
 $Comp
-L GND #PWR0132
+L GND #PWR0135
 U 1 1 5B34DDA4
 P 2550 4950
-F 0 "#PWR0132" H 2550 4700 50  0001 C CNN
+F 0 "#PWR0135" H 2550 4700 50  0001 C CNN
 F 1 "GND" H 2550 4800 50  0000 C CNN
 F 2 "" H 2550 4950 50  0001 C CNN
@@
 $EndComp
 $Comp
-L GND #PWR0133
+L GND #PWR0136
 U 1 1 5B34DE03
 P 3050 4950
-F 0 "#PWR0133" H 3050 4700 50  0001 C CNN
+F 0 "#PWR0136" H 3050 4700 50  0001 C CNN
 F 1 "GND" H 3050 4800 50  0000 C CNN
 F 2 "" H 3050 4950 50  0001 C CNN
@@
 Connection ~ 2850 5600
 $Comp
-L DMG1026UV-7 Q14
-U 2 1 5B356663
-P 4000 6300
-F 0 "Q14" H 4200 6375 50  0000 L CNN
-F 1 "DMG1026UV-7" H 4200 6300 50  0000 L CNN
-F 2 "digikey-footprints:SOT-563" H 4200 6225 50  0001 L CIN
-F 3 "" H 4000 6300 50  0001 L CNN
-	2    4000 6300
-	1    0    0    -1
-$EndComp
-$Comp
-L GND #PWR0134
-U 1 1 5B3566ED
-P 4100 6650
-F 0 "#PWR0134" H 4100 6400 50  0001 C CNN
-F 1 "GND" H 4100 6500 50  0000 C CNN
-F 2 "" H 4100 6650 50  0001 C CNN
-F 3 "" H 4100 6650 50  0001 C CNN
-	1    4100 6650
-	1    0    0    -1
-$EndComp
-Wire Wire Line
-	4100 6500 4100 6650
-Wire Wire Line
-	4100 6100 4100 5850
-Wire Wire Line
-	4100 5850 4900 5850
-Wire Wire Line
-	4900 5850 4900 6600
-Wire Wire Line
-	4900 6600 3650 6600
-Connection ~ 4100 6600
-Wire Wire Line
-	3800 6350 3650 6350
-Wire Wire Line
-	3650 6350 3650 6600
-Text Notes 5100 6300 0    60   ~ 0
-Unused gate
+L 2N7002 Q4
+U 1 1 5BF592AF
+P 2750 6250
+F 0 "Q4" H 2950 6325 50  0000 L CNN
+F 1 "2N7002" H 2950 6250 50  0000 L CNN
+F 2 "TO_SOT_Packages_SMD:SOT-23" H 2950 6175 50  0001 L CIN
+F 3 "" H 2750 6250 50  0001 L CNN
+	1    2750 6250
+	1    0    0    -1
+$EndComp
 $EndSCHEMATC
